File: hardware/finder.sch (KiCad schematic (older format))
At the start: 13 parts, among them U4 TCA9545A, U5 VL6180X_POLOLU, U6 VL6180X_POLOLU, U7 VL6180X_POLOLU, U8 VL6180X_POLOLU

Commit message: updated PCB design
Parts:
- C_RANGE1: footprint (none) -> Capacitors_SMD:C_0603_HandSoldering
- R_RANGE1, R_RANGE2, R_RANGE3, R_RANGE4, R_RANGE5, R_RANGE6, R_RANGE7: footprint (none) -> Resistors_SMD:R_0603_HandSoldering
- U4: footprint (none) -> Housings_SSOP:TSSOP-20_4.4x6.5mm_Pitch0.65mm
- U5, U6, U7, U8: footprint (none) -> footprints_micromouse:VL6180X_POLOLU_Pin_Header_Straight_1x07
Changed lines of the file:
@@
 F 0 "U5" H 6850 2000 60  0000 C CNN
 F 1 "VL6180X_POLOLU" H 7050 1100 60  0000 C CNN
-F 2 "" H 7050 1750 60  0000 C CNN
+F 2 "footprints_micromouse:VL6180X_POLOLU_Pin_Header_Straight_1x07" H 7050 1750 60  0001 C CNN
 F 3 "" H 7050 1750 60  0000 C CNN
 	1    7000 1550
@@
 F 0 "U7" H 8100 3150 60  0000 C CNN
 F 1 "VL6180X_POLOLU" H 8300 2250 60  0000 C CNN
-F 2 "" H 8300 2900 60  0000 C CNN
+F 2 "footprints_micromouse:VL6180X_POLOLU_Pin_Header_Straight_1x07" H 8300 2900 60  0001 C CNN
 F 3 "" H 8300 2900 60  0000 C CNN
 	1    8250 2700
@@
 F 0 "U8" H 8100 4900 60  0000 C CNN
 F 1 "VL6180X_POLOLU" H 8300 4000 60  0000 C CNN
-F 2 "" H 8300 4650 60  0000 C CNN
+F 2 "footprints_micromouse:VL6180X_POLOLU_Pin_Header_Straight_1x07" H 8300 4650 60  0001 C CNN
 F 3 "" H 8300 4650 60  0000 C CNN
 	1    8250 4450
@@
 F 0 "U6" H 7000 6050 60  0000 C CNN
 F 1 "VL6180X_POLOLU" H 7200 5150 60  0000 C CNN
-F 2 "" H 7200 5800 60  0000 C CNN
+F 2 "footprints_micromouse:VL6180X_POLOLU_Pin_Header_Straight_1x07" H 7200 5800 60  0001 C CNN
 F 3 "" H 7200 5800 60  0000 C CNN
 	1    7150 5600
@@
 F 0 "U4" H 4700 4500 60  0000 C CNN
 F 1 "TCA9545A" H 4850 3100 60  0000 C CNN
-F 2 "" H 5050 4200 60  0000 C CNN
+F 2 "Housings_SSOP:TSSOP-20_4.4x6.5mm_Pitch0.65mm" H 5050 4200 60  0001 C CNN
 F 3 "" H 5050 4200 60  0000 C CNN
 	1    5000 3750
@@
 $EndComp
 $Comp
-L +3.3V #PWR15
+L +3.3V #PWR046
 U 1 1 56EB7092
 P 5000 2300
-F 0 "#PWR15" H 5000 2150 50  0001 C CNN
+F 0 "#PWR046" H 5000 2150 50  0001 C CNN
 F 1 "+3.3V" H 5000 2440 50  0000 C CNN
 F 2 "" H 5000 2300 50  0000 C CNN
@@
 $EndComp
 $Comp
-L GND #PWR14
+L GND #PWR047
 U 1 1 56EB70B0
 P 4350 4350
-F 0 "#PWR14" H 4350 4100 50  0001 C CNN
+F 0 "#PWR047" H 4350 4100 50  0001 C CNN
 F 1 "GND" H 4350 4200 50  0000 C CNN
 F 2 "" H 4350 4350 50  0000 C CNN
@@
 $EndComp
 $Comp
-L GND #PWR18
+L GND #PWR048
 U 1 1 56EB7672
 P 7050 2150
-F 0 "#PWR18" H 7050 1900 50  0001 C CNN
+F 0 "#PWR048" H 7050 1900 50  0001 C CNN
 F 1 "GND" H 7050 2000 50  0000 C CNN
 F 2 "" H 7050 2150 50  0000 C CNN
@@
 $EndComp
 $Comp
-L GND #PWR23
+L GND #PWR049
 U 1 1 56EB7690
 P 8300 3300
-F 0 "#PWR23" H 8300 3050 50  0001 C CNN
+F 0 "#PWR049" H 8300 3050 50  0001 C CNN
 F 1 "GND" H 8300 3150 50  0000 C CNN
 F 2 "" H 8300 3300 50  0000 C CNN
@@
 $EndComp
 $Comp
-L GND #PWR24
+L GND #PWR050
 U 1 1 56EB76FD
 P 8300 5050
-F 0 "#PWR24" H 8300 4800 50  0001 C CNN
+F 0 "#PWR050" H 8300 4800 50  0001 C CNN
 F 1 "GND" H 8300 4900 50  0000 C CNN
 F 2 "" H 8300 5050 50  0000 C CNN
@@
 $EndComp
 $Comp
-L GND #PWR20
+L GND #PWR051
 U 1 1 56EB7739
 P 7200 6200
-F 0 "#PWR20" H 7200 5950 50  0001 C CNN
+F 0 "#PWR051" H 7200 5950 50  0001 C CNN
 F 1 "GND" H 7200 6050 50  0000 C CNN
 F 2 "" H 7200 6200 50  0000 C CNN
@@
 $EndComp
 $Comp
-L +3.3V #PWR21
+L +3.3V #PWR052
 U 1 1 56EB79E4
 P 8250 2100
-F 0 "#PWR21" H 8250 1950 50  0001 C CNN
+F 0 "#PWR052" H 8250 1950 50  0001 C CNN
 F 1 "+3.3V" H 8250 2240 50  0000 C CNN
 F 2 "" H 8250 2100 50  0000 C CNN
@@
 $EndComp
 $Comp
-L +3.3V #PWR22
+L +3.3V #PWR053
 U 1 1 56EB7A02
 P 8250 3850
-F 0 "#PWR22" H 8250 3700 50  0001 C CNN
+F 0 "#PWR053" H 8250 3700 50  0001 C CNN
 F 1 "+3.3V" H 8250 3990 50  0000 C CNN
 F 2 "" H 8250 3850 50  0000 C CNN
@@
 $EndComp
 $Comp
-L +3.3V #PWR19
+L +3.3V #PWR054
 U 1 1 56EB7A20
 P 7150 5000
-F 0 "#PWR19" H 7150 4850 50  0001 C CNN
+F 0 "#PWR054" H 7150 4850 50  0001 C CNN
 F 1 "+3.3V" H 7150 5140 50  0000 C CNN
 F 2 "" H 7150 5000 50  0000 C CNN
@@
 $EndComp
 $Comp
-L +3.3V #PWR17
+L +3.3V #PWR055
 U 1 1 56EB7A5C
 P 7000 950
-F 0 "#PWR17" H 7000 800 50  0001 C CNN
+F 0 "#PWR055" H 7000 800 50  0001 C CNN
 F 1 "+3.3V" H 7000 1090 50  0000 C CNN
 F 2 "" H 7000 950 50  0000 C CNN
@@
 F 0 "R_RANGE4" V 5540 2810 50  0000 L CNN
 F 1 "10k" V 5660 2810 50  0000 L CNN
-F 2 "" H 5600 2900 50  0000 C CNN
+F 2 "Resistors_SMD:R_0603_HandSoldering" H 5600 2900 50  0001 C CNN
 F 3 "" H 5600 2900 50  0000 C CNN
 	1    5600 2900
@@
 F 0 "R_RANGE5" V 5740 2810 50  0000 L CNN
 F 1 "10k" V 5860 2810 50  0000 L CNN
-F 2 "" H 5800 2900 50  0000 C CNN
+F 2 "Resistors_SMD:R_0603_HandSoldering" H 5800 2900 50  0001 C CNN
 F 3 "" H 5800 2900 50  0000 C CNN
 	1    5800 2900
@@
 F 0 "R_RANGE6" V 5940 2810 50  0000 L CNN
 F 1 "10k" V 6060 2810 50  0000 L CNN
-F 2 "" H 6000 2900 50  0000 C CNN
+F 2 "Resistors_SMD:R_0603_HandSoldering" H 6000 2900 50  0001 C CNN
 F 3 "" H 6000 2900 50  0000 C CNN
 	1    6000 2900
@@
 F 0 "R_RANGE7" V 6140 2810 50  0000 L CNN
 F 1 "10k" V 6260 2810 50  0000 L CNN
-F 2 "" H 6200 2900 50  0000 C CNN
+F 2 "Resistors_SMD:R_0603_HandSoldering" H 6200 2900 50  0001 C CNN
 F 3 "" H 6200 2900 50  0000 C CNN
 	1    6200 2900
@@
 F 0 "R_RANGE3" V 4240 2810 50  0000 L CNN
 F 1 "10k" V 4360 2810 50  0000 L CNN
-F 2 "" H 4300 2900 50  0000 C CNN
+F 2 "Resistors_SMD:R_0603_HandSoldering" H 4300 2900 50  0001 C CNN
 F 3 "" H 4300 2900 50  0000 C CNN
 	1    4300 2900
@@
 F 0 "R_RANGE2" V 4040 2810 50  0000 L CNN
 F 1 "10k" V 4160 2810 50  0000 L CNN
-F 2 "" H 4100 2900 50  0000 C CNN
+F 2 "Resistors_SMD:R_0603_HandSoldering" H 4100 2900 50  0001 C CNN
 F 3 "" H 4100 2900 50  0000 C CNN
 	1    4100 2900
@@
 F 0 "R_RANGE1" V 3840 2810 50  0000 L CNN
 F 1 "10k" V 3960 2810 50  0000 L CNN
-F 2 "" H 3900 2900 50  0000 C CNN
+F 2 "Resistors_SMD:R_0603_HandSoldering" H 3900 2900 50  0001 C CNN
 F 3 "" H 3900 2900 50  0000 C CNN
 	1    3900 2900
@@
 F 0 "C_RANGE1" H 5510 2270 50  0000 L CNN
 F 1 "0.1uF" H 5520 2120 50  0000 L CNN
-F 2 "" H 5500 2200 50  0000 C CNN
+F 2 "Capacitors_SMD:C_0603_HandSoldering" H 5500 2200 50  0001 C CNN
 F 3 "" H 5500 2200 50  0000 C CNN
 	1    5500 2200
@@
 Connection ~ 5000 2400
 $Comp
-L GND #PWR16
+L GND #PWR056
 U 1 1 56ED580E
 P 5500 2350
-F 0 "#PWR16" H 5500 2100 50  0001 C CNN
+F 0 "#PWR056" H 5500 2100 50  0001 C CNN
 F 1 "GND" H 5500 2200 50  0000 C CNN
 F 2 "" H 5500 2350 50  0000 C CNN

Commit message: PCB board- needs to check the motor driver
Parts:
- C_RANGE1: footprint Capacitors_SMD:C_0603_HandSoldering -> Capacitors_SMD:C_0603
- R_RANGE1, R_RANGE2, R_RANGE3, R_RANGE4, R_RANGE5, R_RANGE6, R_RANGE7: footprint Resistors_SMD:R_0603_HandSoldering -> Resistors_SMD:R_0603
Changed lines of the file:
@@
 $EndComp
 $Comp
-L +3.3V #PWR046
+L +3.3V #PWR049
 U 1 1 56EB7092
 P 5000 2300
-F 0 "#PWR046" H 5000 2150 50  0001 C CNN
+F 0 "#PWR049" H 5000 2150 50  0001 C CNN
 F 1 "+3.3V" H 5000 2440 50  0000 C CNN
 F 2 "" H 5000 2300 50  0000 C CNN
@@
 $EndComp
 $Comp
-L GND #PWR047
+L GND #PWR050
 U 1 1 56EB70B0
 P 4350 4350
-F 0 "#PWR047" H 4350 4100 50  0001 C CNN
+F 0 "#PWR050" H 4350 4100 50  0001 C CNN
 F 1 "GND" H 4350 4200 50  0000 C CNN
 F 2 "" H 4350 4350 50  0000 C CNN
@@
 $EndComp
 $Comp
-L GND #PWR048
+L GND #PWR051
 U 1 1 56EB7672
 P 7050 2150
-F 0 "#PWR048" H 7050 1900 50  0001 C CNN
+F 0 "#PWR051" H 7050 1900 50  0001 C CNN
 F 1 "GND" H 7050 2000 50  0000 C CNN
 F 2 "" H 7050 2150 50  0000 C CNN
@@
 $EndComp
 $Comp
-L GND #PWR049
+L GND #PWR052
 U 1 1 56EB7690
 P 8300 3300
-F 0 "#PWR049" H 8300 3050 50  0001 C CNN
+F 0 "#PWR052" H 8300 3050 50  0001 C CNN
 F 1 "GND" H 8300 3150 50  0000 C CNN
 F 2 "" H 8300 3300 50  0000 C CNN
@@
 $EndComp
 $Comp
-L GND #PWR050
+L GND #PWR053
 U 1 1 56EB76FD
 P 8300 5050
-F 0 "#PWR050" H 8300 4800 50  0001 C CNN
+F 0 "#PWR053" H 8300 4800 50  0001 C CNN
 F 1 "GND" H 8300 4900 50  0000 C CNN
 F 2 "" H 8300 5050 50  0000 C CNN
@@
 $EndComp
 $Comp
-L GND #PWR051
+L GND #PWR054
 U 1 1 56EB7739
 P 7200 6200
-F 0 "#PWR051" H 7200 5950 50  0001 C CNN
+F 0 "#PWR054" H 7200 5950 50  0001 C CNN
 F 1 "GND" H 7200 6050 50  0000 C CNN
 F 2 "" H 7200 6200 50  0000 C CNN
@@
 $EndComp
 $Comp
-L +3.3V #PWR052
+L +3.3V #PWR055
 U 1 1 56EB79E4
 P 8250 2100
-F 0 "#PWR052" H 8250 1950 50  0001 C CNN
+F 0 "#PWR055" H 8250 1950 50  0001 C CNN
 F 1 "+3.3V" H 8250 2240 50  0000 C CNN
 F 2 "" H 8250 2100 50  0000 C CNN
@@
 $EndComp
 $Comp
-L +3.3V #PWR053
+L +3.3V #PWR056
 U 1 1 56EB7A02
 P 8250 3850
-F 0 "#PWR053" H 8250 3700 50  0001 C CNN
+F 0 "#PWR056" H 8250 3700 50  0001 C CNN
 F 1 "+3.3V" H 8250 3990 50  0000 C CNN
 F 2 "" H 8250 3850 50  0000 C CNN
@@
 $EndComp
 $Comp
-L +3.3V #PWR054
+L +3.3V #PWR057
 U 1 1 56EB7A20
 P 7150 5000
-F 0 "#PWR054" H 7150 4850 50  0001 C CNN
+F 0 "#PWR057" H 7150 4850 50  0001 C CNN
 F 1 "+3.3V" H 7150 5140 50  0000 C CNN
 F 2 "" H 7150 5000 50  0000 C CNN
@@
 $EndComp
 $Comp
-L +3.3V #PWR055
+L +3.3V #PWR058
 U 1 1 56EB7A5C
 P 7000 950
-F 0 "#PWR055" H 7000 800 50  0001 C CNN
+F 0 "#PWR058" H 7000 800 50  0001 C CNN
 F 1 "+3.3V" H 7000 1090 50  0000 C CNN
 F 2 "" H 7000 950 50  0000 C CNN
@@
 F 0 "R_RANGE4" V 5540 2810 50  0000 L CNN
 F 1 "10k" V 5660 2810 50  0000 L CNN
-F 2 "Resistors_SMD:R_0603_HandSoldering" H 5600 2900 50  0001 C CNN
+F 2 "Resistors_SMD:R_0603" H 5600 2900 50  0001 C CNN
 F 3 "" H 5600 2900 50  0000 C CNN
 	1    5600 2900
@@
 F 0 "R_RANGE5" V 5740 2810 50  0000 L CNN
 F 1 "10k" V 5860 2810 50  0000 L CNN
-F 2 "Resistors_SMD:R_0603_HandSoldering" H 5800 2900 50  0001 C CNN
+F 2 "Resistors_SMD:R_0603" H 5800 2900 50  0001 C CNN
 F 3 "" H 5800 2900 50  0000 C CNN
 	1    5800 2900
@@
 F 0 "R_RANGE6" V 5940 2810 50  0000 L CNN
 F 1 "10k" V 6060 2810 50  0000 L CNN
-F 2 "Resistors_SMD:R_0603_HandSoldering" H 6000 2900 50  0001 C CNN
+F 2 "Resistors_SMD:R_0603" H 6000 2900 50  0001 C CNN
 F 3 "" H 6000 2900 50  0000 C CNN
 	1    6000 2900
@@
 F 0 "R_RANGE7" V 6140 2810 50  0000 L CNN
 F 1 "10k" V 6260 2810 50  0000 L CNN
-F 2 "Resistors_SMD:R_0603_HandSoldering" H 6200 2900 50  0001 C CNN
+F 2 "Resistors_SMD:R_0603" H 6200 2900 50  0001 C CNN
 F 3 "" H 6200 2900 50  0000 C CNN
 	1    6200 2900
@@
 F 0 "R_RANGE3" V 4240 2810 50  0000 L CNN
 F 1 "10k" V 4360 2810 50  0000 L CNN
-F 2 "Resistors_SMD:R_0603_HandSoldering" H 4300 2900 50  0001 C CNN
+F 2 "Resistors_SMD:R_0603" H 4300 2900 50  0001 C CNN
 F 3 "" H 4300 2900 50  0000 C CNN
 	1    4300 2900
@@
 F 0 "R_RANGE2" V 4040 2810 50  0000 L CNN
 F 1 "10k" V 4160 2810 50  0000 L CNN
-F 2 "Resistors_SMD:R_0603_HandSoldering" H 4100 2900 50  0001 C CNN
+F 2 "Resistors_SMD:R_0603" H 4100 2900 50  0001 C CNN
 F 3 "" H 4100 2900 50  0000 C CNN
 	1    4100 2900
@@
 F 0 "R_RANGE1" V 3840 2810 50  0000 L CNN
 F 1 "10k" V 3960 2810 50  0000 L CNN
-F 2 "Resistors_SMD:R_0603_HandSoldering" H 3900 2900 50  0001 C CNN
+F 2 "Resistors_SMD:R_0603" H 3900 2900 50  0001 C CNN
 F 3 "" H 3900 2900 50  0000 C CNN
 	1    3900 2900
@@
 F 0 "C_RANGE1" H 5510 2270 50  0000 L CNN
 F 1 "0.1uF" H 5520 2120 50  0000 L CNN
-F 2 "Capacitors_SMD:C_0603_HandSoldering" H 5500 2200 50  0001 C CNN
+F 2 "Capacitors_SMD:C_0603" H 5500 2200 50  0001 C CNN
 F 3 "" H 5500 2200 50  0000 C CNN
 	1    5500 2200
@@
 Connection ~ 5000 2400
 $Comp
-L GND #PWR056
+L GND #PWR059
 U 1 1 56ED580E
 P 5500 2350
-F 0 "#PWR056" H 5500 2100 50  0001 C CNN
+F 0 "#PWR059" H 5500 2100 50  0001 C CNN
 F 1 "GND" H 5500 2200 50  0000 C CNN
 F 2 "" H 5500 2350 50  0000 C CNN
