File: hardware/uSD_IMU_DIS.sch (KiCad schematic (older format))
At the start: 13 parts, among them J1 uSD_SLOT_47219-2001, U10 MPU-9250, U9 HCMS-2901

Commit message: updated PCB design
Parts:
- C_DIS1, C_IMU1, C_IMU3: footprint (none) -> Capacitors_SMD:C_0603_HandSoldering
- C_DIS2, C_uSD1: footprint (none) -> Capacitors_SMD:C_1206_HandSoldering
- C_IMU2: footprint (none) -> Capacitors_SMD:C_0805_HandSoldering
- D1: footprint (none) -> LEDs:LED_0603
- J1: footprint uSD_SLOT_47219-2001 -> footprints_micromouse:uSD_MOLEX_47219-2001
- R_IMU1, R_IMU2, R_uSD1: footprint (none) -> Resistors_SMD:R_0603_HandSoldering
- U10: footprint QFN-24/3MM -> MPU-9250:QFN-24%2f3MM
- U9: footprint HCMS-2901 -> footprints_micromouse:HCMS-2903
Changed lines of the file:
@@
 F 0 "U9" H 3050 6450 45  0000 C CNN
 F 1 "HCMS-2901" H 3400 6450 45  0000 C CNN
-F 2 "HCMS-2901" H 3500 5650 20  0001 C CNN
+F 2 "footprints_micromouse:HCMS-2903" H 3500 5650 20  0001 C CNN
 F 3 "" H 3300 6050 60  0000 C CNN
 	1    3300 6050
@@
 F 0 "U10" H 3000 3800 50  0000 L CNN
 F 1 "MPU-9250" H 2800 2800 50  0000 L CNN
-F 2 "QFN-24/3MM" H 3600 2800 50  0001 L CNN
+F 2 "MPU-9250:QFN-24%2f3MM" H 3600 2800 50  0001 L CNN
 F 3 "" H 3400 3250 60  0000 C CNN
 	1    3400 3250
@@
 F 0 "J1" H 7950 4450 50  0000 L CNN
 F 1 "uSD_SLOT_47219-2001" H 7950 4350 50  0000 L CNN
-F 2 "uSD_SLOT_47219-2001" H 7950 3450 50  0001 L CNN
+F 2 "footprints_micromouse:uSD_MOLEX_47219-2001" H 7950 3450 50  0001 L CNN
 F 3 "" H 8450 3900 60  0000 C CNN
 	1    8450 3900
@@
 $EndComp
 $Comp
-L +3.3V #PWR35
+L +3.3V #PWR057
 U 1 1 56EC0B54
 P 9300 3450
-F 0 "#PWR35" H 9300 3300 50  0001 C CNN
+F 0 "#PWR057" H 9300 3300 50  0001 C CNN
 F 1 "+3.3V" H 9300 3590 50  0000 C CNN
 F 2 "" H 9300 3450 50  0000 C CNN
@@
 $EndComp
 $Comp
-L GND #PWR36
+L GND #PWR058
 U 1 1 56EC0C8A
 P 9300 4250
-F 0 "#PWR36" H 9300 4000 50  0001 C CNN
+F 0 "#PWR058" H 9300 4000 50  0001 C CNN
 F 1 "GND" H 9300 4100 50  0000 C CNN
 F 2 "" H 9300 4250 50  0000 C CNN
@@
 F 0 "C_DIS1" H 4110 6120 50  0000 L CNN
 F 1 "0.1uF" H 4110 5970 50  0000 L CNN
-F 2 "" H 4100 6050 50  0000 C CNN
+F 2 "Capacitors_SMD:C_0603_HandSoldering" H 4100 6050 50  0001 C CNN
 F 3 "" H 4100 6050 50  0000 C CNN
 	1    4100 6050
@@
 $EndComp
 $Comp
-L +5V #PWR32
+L +5V #PWR059
 U 1 1 56EC13E1
 P 4100 5550
-F 0 "#PWR32" H 4100 5400 50  0001 C CNN
+F 0 "#PWR059" H 4100 5400 50  0001 C CNN
 F 1 "+5V" H 4100 5690 50  0000 C CNN
 F 2 "" H 4100 5550 50  0000 C CNN
@@
 	3800 6200 4450 6200
 $Comp
-L GND #PWR33
+L GND #PWR060
 U 1 1 56EC150D
 P 4100 6550
-F 0 "#PWR33" H 4100 6300 50  0001 C CNN
+F 0 "#PWR060" H 4100 6300 50  0001 C CNN
 F 1 "GND" H 4100 6400 50  0000 C CNN
 F 2 "" H 4100 6550 50  0000 C CNN
@@
 F 0 "C_DIS2" H 4460 6120 50  0000 L CNN
 F 1 "10uF" H 4460 5970 50  0000 L CNN
-F 2 "" H 4450 6050 50  0000 C CNN
+F 2 "Capacitors_SMD:C_1206_HandSoldering" H 4450 6050 50  0001 C CNN
 F 3 "" H 4450 6050 50  0000 C CNN
 	1    4450 6050
@@
 	4450 6200 4450 6150
 $Comp
-L +5V #PWR26
+L +5V #PWR061
 U 1 1 56EC1816
 P 2350 5800
-F 0 "#PWR26" H 2350 5650 50  0001 C CNN
+F 0 "#PWR061" H 2350 5650 50  0001 C CNN
 F 1 "+5V" H 2350 5940 50  0000 C CNN
 F 2 "" H 2350 5800 50  0000 C CNN
@@
 F 0 "D1" H 7300 4825 50  0000 L CNN
 F 1 "Led_Small" H 7175 4600 50  0001 L CNN
-F 2 "" V 7350 4700 50  0000 C CNN
+F 2 "LEDs:LED_0603" V 7350 4700 50  0001 C CNN
 F 3 "" V 7350 4700 50  0000 C CNN
 	1    7350 4700
@@
 F 0 "R_uSD1" H 7680 4720 50  0000 L CNN
 F 1 "1k" H 7680 4660 50  0000 L CNN
-F 2 "" H 7650 4700 50  0000 C CNN
+F 2 "Resistors_SMD:R_0603_HandSoldering" H 7650 4700 50  0001 C CNN
 F 3 "" H 7650 4700 50  0000 C CNN
 	1    7650 4700
@@
 Connection ~ 7700 4200
 $Comp
-L GND #PWR28
+L GND #PWR062
 U 1 1 56EC2E0A
 P 3450 4050
-F 0 "#PWR28" H 3450 3800 50  0001 C CNN
+F 0 "#PWR062" H 3450 3800 50  0001 C CNN
 F 1 "GND" H 3450 3900 50  0000 C CNN
 F 2 "" H 3450 4050 50  0000 C CNN
@@
 Connection ~ 3450 3900
 $Comp
-L +3.3V #PWR29
+L +3.3V #PWR063
 U 1 1 56EC3332
 P 3500 2100
-F 0 "#PWR29" H 3500 1950 50  0001 C CNN
+F 0 "#PWR063" H 3500 1950 50  0001 C CNN
 F 1 "+3.3V" H 3500 2240 50  0000 C CNN
 F 2 "" H 3500 2100 50  0000 C CNN
@@
 F 0 "C_IMU1" H 2310 3370 50  0000 L CNN
 F 1 "0.1uF" H 2320 3220 50  0000 L CNN
-F 2 "" H 2300 3300 50  0000 C CNN
+F 2 "Capacitors_SMD:C_0603_HandSoldering" H 2300 3300 50  0001 C CNN
 F 3 "" H 2300 3300 50  0000 C CNN
 	1    2300 3300
@@
 	2300 3150 2300 3200
 $Comp
-L GND #PWR25
+L GND #PWR064
 U 1 1 56EC3E3A
 P 2300 3550
-F 0 "#PWR25" H 2300 3300 50  0001 C CNN
+F 0 "#PWR064" H 2300 3300 50  0001 C CNN
 F 1 "GND" H 2300 3400 50  0000 C CNN
 F 2 "" H 2300 3550 50  0000 C CNN
@@
 F 0 "C_IMU3" H 4060 2470 50  0000 L CNN
 F 1 "0.1uF" H 4070 2320 50  0000 L CNN
-F 2 "" H 4050 2400 50  0000 C CNN
+F 2 "Capacitors_SMD:C_0603_HandSoldering" H 4050 2400 50  0001 C CNN
 F 3 "" H 4050 2400 50  0000 C CNN
 	1    4050 2400
@@
 F 0 "C_IMU2" H 3710 2470 50  0000 L CNN
 F 1 "10nF" H 3720 2320 50  0000 L CNN
-F 2 "" H 3700 2400 50  0000 C CNN
+F 2 "Capacitors_SMD:C_0805_HandSoldering" H 3700 2400 50  0001 C CNN
 F 3 "" H 3700 2400 50  0000 C CNN
 	1    3700 2400
@@
 	4050 2500 4050 2700
 $Comp
-L GND #PWR30
+L GND #PWR065
 U 1 1 56EC45CA
 P 4050 2700
-F 0 "#PWR30" H 4050 2450 50  0001 C CNN
+F 0 "#PWR065" H 4050 2450 50  0001 C CNN
 F 1 "GND" H 4050 2550 50  0000 C CNN
 F 2 "" H 4050 2700 50  0000 C CNN
@@
 	3900 3400 4100 3400
 $Comp
-L GND #PWR31
+L GND #PWR066
 U 1 1 56EC4DCF
 P 4100 4050
-F 0 "#PWR31" H 4100 3800 50  0001 C CNN
+F 0 "#PWR066" H 4100 3800 50  0001 C CNN
 F 1 "GND" H 4100 3900 50  0000 C CNN
 F 2 "" H 4100 4050 50  0000 C CNN
@@
 F 0 "R_IMU2" V 4590 2760 50  0000 L CNN
 F 1 "10k" V 4710 2760 50  0000 L CNN
-F 2 "" H 4650 2850 50  0000 C CNN
+F 2 "Resistors_SMD:R_0603_HandSoldering" H 4650 2850 50  0001 C CNN
 F 3 "" H 4650 2850 50  0000 C CNN
 	1    4650 2850
@@
 F 0 "R_IMU1" V 4390 2760 50  0000 L CNN
 F 1 "10k" V 4510 2760 50  0000 L CNN
-F 2 "" H 4450 2850 50  0000 C CNN
+F 2 "Resistors_SMD:R_0603_HandSoldering" H 4450 2850 50  0001 C CNN
 F 3 "" H 4450 2850 50  0000 C CNN
 	1    4450 2850
@@
 $EndComp
 $Comp
-L +3.3V #PWR34
+L +3.3V #PWR067
 U 1 1 56EC6F0F
 P 4650 2500
-F 0 "#PWR34" H 4650 2350 50  0001 C CNN
+F 0 "#PWR067" H 4650 2350 50  0001 C CNN
 F 1 "+3.3V" H 4650 2640 50  0000 C CNN
 F 2 "" H 4650 2500 50  0000 C CNN
@@
 F 0 "C_uSD1" H 9560 3970 50  0000 L CNN
 F 1 "10uF" H 9570 3820 50  0000 L CNN
-F 2 "" H 9550 3900 50  0000 C CNN
+F 2 "Capacitors_SMD:C_1206_HandSoldering" H 9550 3900 50  0001 C CNN
 F 3 "" H 9550 3900 50  0000 C CNN
 	1    9550 3900
@@
 	9550 4200 9550 4000
 $Comp
-L GND #PWR27
+L GND #PWR068
 U 1 1 56EDA0C0
 P 2650 3700
-F 0 "#PWR27" H 2650 3450 50  0001 C CNN
+F 0 "#PWR068" H 2650 3450 50  0001 C CNN
 F 1 "GND" H 2650 3550 50  0000 C CNN
 F 2 "" H 2650 3700 50  0000 C CNN

Commit message: PCB board- needs to check the motor driver
Parts:
- C_DIS1, C_IMU1, C_IMU3: footprint Capacitors_SMD:C_0603_HandSoldering -> Capacitors_SMD:C_0603
- C_DIS2, C_uSD1: footprint Capacitors_SMD:C_1206_HandSoldering -> Capacitors_SMD:C_1206
- C_IMU2: footprint Capacitors_SMD:C_0805_HandSoldering -> Capacitors_SMD:C_0805
- R_IMU1, R_IMU2, R_uSD1: footprint Resistors_SMD:R_0603_HandSoldering -> Resistors_SMD:R_0603
- U10: footprint MPU-9250:QFN-24%2f3MM -> footprints_micromouse:MPU-9250
Changed lines of the file:
@@
 F 0 "U10" H 3000 3800 50  0000 L CNN
 F 1 "MPU-9250" H 2800 2800 50  0000 L CNN
-F 2 "MPU-9250:QFN-24%2f3MM" H 3600 2800 50  0001 L CNN
+F 2 "footprints_micromouse:MPU-9250" H 3600 2800 50  0001 L CNN
 F 3 "" H 3400 3250 60  0000 C CNN
 	1    3400 3250
@@
 $EndComp
 $Comp
-L +3.3V #PWR057
+L +3.3V #PWR060
 U 1 1 56EC0B54
 P 9300 3450
-F 0 "#PWR057" H 9300 3300 50  0001 C CNN
+F 0 "#PWR060" H 9300 3300 50  0001 C CNN
 F 1 "+3.3V" H 9300 3590 50  0000 C CNN
 F 2 "" H 9300 3450 50  0000 C CNN
@@
 $EndComp
 $Comp
-L GND #PWR058
+L GND #PWR061
 U 1 1 56EC0C8A
 P 9300 4250
-F 0 "#PWR058" H 9300 4000 50  0001 C CNN
+F 0 "#PWR061" H 9300 4000 50  0001 C CNN
 F 1 "GND" H 9300 4100 50  0000 C CNN
 F 2 "" H 9300 4250 50  0000 C CNN
@@
 F 0 "C_DIS1" H 4110 6120 50  0000 L CNN
 F 1 "0.1uF" H 4110 5970 50  0000 L CNN
-F 2 "Capacitors_SMD:C_0603_HandSoldering" H 4100 6050 50  0001 C CNN
+F 2 "Capacitors_SMD:C_0603" H 4100 6050 50  0001 C CNN
 F 3 "" H 4100 6050 50  0000 C CNN
 	1    4100 6050
@@
 $EndComp
 $Comp
-L +5V #PWR059
+L +5V #PWR062
 U 1 1 56EC13E1
 P 4100 5550
-F 0 "#PWR059" H 4100 5400 50  0001 C CNN
+F 0 "#PWR062" H 4100 5400 50  0001 C CNN
 F 1 "+5V" H 4100 5690 50  0000 C CNN
 F 2 "" H 4100 5550 50  0000 C CNN
@@
 	3800 6200 4450 6200
 $Comp
-L GND #PWR060
+L GND #PWR063
 U 1 1 56EC150D
 P 4100 6550
-F 0 "#PWR060" H 4100 6300 50  0001 C CNN
+F 0 "#PWR063" H 4100 6300 50  0001 C CNN
 F 1 "GND" H 4100 6400 50  0000 C CNN
 F 2 "" H 4100 6550 50  0000 C CNN
@@
 F 0 "C_DIS2" H 4460 6120 50  0000 L CNN
 F 1 "10uF" H 4460 5970 50  0000 L CNN
-F 2 "Capacitors_SMD:C_1206_HandSoldering" H 4450 6050 50  0001 C CNN
+F 2 "Capacitors_SMD:C_1206" H 4450 6050 50  0001 C CNN
 F 3 "" H 4450 6050 50  0000 C CNN
 	1    4450 6050
@@
 	4450 6200 4450 6150
 $Comp
-L +5V #PWR061
+L +5V #PWR064
 U 1 1 56EC1816
 P 2350 5800
-F 0 "#PWR061" H 2350 5650 50  0001 C CNN
+F 0 "#PWR064" H 2350 5650 50  0001 C CNN
 F 1 "+5V" H 2350 5940 50  0000 C CNN
 F 2 "" H 2350 5800 50  0000 C CNN
@@
 F 0 "R_uSD1" H 7680 4720 50  0000 L CNN
 F 1 "1k" H 7680 4660 50  0000 L CNN
-F 2 "Resistors_SMD:R_0603_HandSoldering" H 7650 4700 50  0001 C CNN
+F 2 "Resistors_SMD:R_0603" H 7650 4700 50  0001 C CNN
 F 3 "" H 7650 4700 50  0000 C CNN
 	1    7650 4700
@@
 Connection ~ 7700 4200
 $Comp
-L GND #PWR062
+L GND #PWR065
 U 1 1 56EC2E0A
 P 3450 4050
-F 0 "#PWR062" H 3450 3800 50  0001 C CNN
+F 0 "#PWR065" H 3450 3800 50  0001 C CNN
 F 1 "GND" H 3450 3900 50  0000 C CNN
 F 2 "" H 3450 4050 50  0000 C CNN
@@
 Connection ~ 3450 3900
 $Comp
-L +3.3V #PWR063
+L +3.3V #PWR066
 U 1 1 56EC3332
 P 3500 2100
-F 0 "#PWR063" H 3500 1950 50  0001 C CNN
+F 0 "#PWR066" H 3500 1950 50  0001 C CNN
 F 1 "+3.3V" H 3500 2240 50  0000 C CNN
 F 2 "" H 3500 2100 50  0000 C CNN
@@
 F 0 "C_IMU1" H 2310 3370 50  0000 L CNN
 F 1 "0.1uF" H 2320 3220 50  0000 L CNN
-F 2 "Capacitors_SMD:C_0603_HandSoldering" H 2300 3300 50  0001 C CNN
+F 2 "Capacitors_SMD:C_0603" H 2300 3300 50  0001 C CNN
 F 3 "" H 2300 3300 50  0000 C CNN
 	1    2300 3300
@@
 	2300 3150 2300 3200
 $Comp
-L GND #PWR064
+L GND #PWR067
 U 1 1 56EC3E3A
 P 2300 3550
-F 0 "#PWR064" H 2300 3300 50  0001 C CNN
+F 0 "#PWR067" H 2300 3300 50  0001 C CNN
 F 1 "GND" H 2300 3400 50  0000 C CNN
 F 2 "" H 2300 3550 50  0000 C CNN
@@
 F 0 "C_IMU3" H 4060 2470 50  0000 L CNN
 F 1 "0.1uF" H 4070 2320 50  0000 L CNN
-F 2 "Capacitors_SMD:C_0603_HandSoldering" H 4050 2400 50  0001 C CNN
+F 2 "Capacitors_SMD:C_0603" H 4050 2400 50  0001 C CNN
 F 3 "" H 4050 2400 50  0000 C CNN
 	1    4050 2400
@@
 F 0 "C_IMU2" H 3710 2470 50  0000 L CNN
 F 1 "10nF" H 3720 2320 50  0000 L CNN
-F 2 "Capacitors_SMD:C_0805_HandSoldering" H 3700 2400 50  0001 C CNN
+F 2 "Capacitors_SMD:C_0805" H 3700 2400 50  0001 C CNN
 F 3 "" H 3700 2400 50  0000 C CNN
 	1    3700 2400
@@
 	4050 2500 4050 2700
 $Comp
-L GND #PWR065
+L GND #PWR068
 U 1 1 56EC45CA
 P 4050 2700
-F 0 "#PWR065" H 4050 2450 50  0001 C CNN
+F 0 "#PWR068" H 4050 2450 50  0001 C CNN
 F 1 "GND" H 4050 2550 50  0000 C CNN
 F 2 "" H 4050 2700 50  0000 C CNN
@@
 	3900 3400 4100 3400
 $Comp
-L GND #PWR066
+L GND #PWR069
 U 1 1 56EC4DCF
 P 4100 4050
-F 0 "#PWR066" H 4100 3800 50  0001 C CNN
+F 0 "#PWR069" H 4100 3800 50  0001 C CNN
 F 1 "GND" H 4100 3900 50  0000 C CNN
 F 2 "" H 4100 4050 50  0000 C CNN
@@
 F 0 "R_IMU2" V 4590 2760 50  0000 L CNN
 F 1 "10k" V 4710 2760 50  0000 L CNN
-F 2 "Resistors_SMD:R_0603_HandSoldering" H 4650 2850 50  0001 C CNN
+F 2 "Resistors_SMD:R_0603" H 4650 2850 50  0001 C CNN
 F 3 "" H 4650 2850 50  0000 C CNN
 	1    4650 2850
@@
 F 0 "R_IMU1" V 4390 2760 50  0000 L CNN
 F 1 "10k" V 4510 2760 50  0000 L CNN
-F 2 "Resistors_SMD:R_0603_HandSoldering" H 4450 2850 50  0001 C CNN
+F 2 "Resistors_SMD:R_0603" H 4450 2850 50  0001 C CNN
 F 3 "" H 4450 2850 50  0000 C CNN
 	1    4450 2850
@@
 $EndComp
 $Comp
-L +3.3V #PWR067
+L +3.3V #PWR070
 U 1 1 56EC6F0F
 P 4650 2500
-F 0 "#PWR067" H 4650 2350 50  0001 C CNN
+F 0 "#PWR070" H 4650 2350 50  0001 C CNN
 F 1 "+3.3V" H 4650 2640 50  0000 C CNN
 F 2 "" H 4650 2500 50  0000 C CNN
@@
 F 0 "C_uSD1" H 9560 3970 50  0000 L CNN
 F 1 "10uF" H 9570 3820 50  0000 L CNN
-F 2 "Capacitors_SMD:C_1206_HandSoldering" H 9550 3900 50  0001 C CNN
+F 2 "Capacitors_SMD:C_1206" H 9550 3900 50  0001 C CNN
 F 3 "" H 9550 3900 50  0000 C CNN
 	1    9550 3900
@@
 	9550 4200 9550 4000
 $Comp
-L GND #PWR068
+L GND #PWR071
 U 1 1 56EDA0C0
 P 2650 3700
-F 0 "#PWR068" H 2650 3450 50  0001 C CNN
+F 0 "#PWR071" H 2650 3450 50  0001 C CNN
 F 1 "GND" H 2650 3550 50  0000 C CNN
 F 2 "" H 2650 3700 50  0000 C CNN
