File: hardware/micromouse.kicad_pcb (KiCad board)
At the start: 2 copper layers, 100 x 74 mm, 79 parts, among them CN1 5_PIN_HEADER, CN2 5_PIN_HEADER, J1 uSD_SLOT_47219-2001, M1 MOTOR_MOUNTS_AND_ENCODERS, M3 2.54MM-SLIDE-SWITCH_TS02_SWIT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, P1 B3B-PH-SM4-TB, P2 B3B-PH-SM4-TB, SW1 SWITCH_DPST, SW2 SWITCH_DPST, SW3 SWITCH_DPST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

Commit message: Fixed the 3.3V line problem of the right corner
Routing:
- net +3V3: track 268.8 -> 266.0 mm
Changed lines of the file:
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@@
     (thickness 1.6)
     (drawings 42)
-    (tracks 1281)
+    (tracks 1282)
     (zones 0)
     (modules 79)
@@
   (page A4)
   (layers
-    (0 F.Cu signal)
+    (0 F.Cu signal hide)
     (31 B.Cu signal)
     (32 B.Adhes user hide)
@@
   )
   (setup
-    (last_trace_width 0.25)
+    (last_trace_width 0.8)
     (user_trace_width 0.2)
     (user_trace_width 0.28)
@@
   (via (at 175.98 93.85) (size 0.6) (drill 0.4) (layers F.Cu B.Cu) (net 5))
   (segment (start 175.879938 93.749938) (end 175.98 93.85) (width 0.28) (layer F.Cu) (net 5))
+  (segment (start 155.5 64) (end 154.75 64) (width 0.8) (layer F.Cu) (net 6))
+  (segment (start 154.75 64) (end 146 72.75) (width 0.8) (layer F.Cu) (net 6))
   (segment (start 218 96.25) (end 216.26 96.25) (width 0.4) (layer F.Cu) (net 6))
   (segment (start 219.75 92.76) (end 219.75 89.5) (width 0.4) (layer B.Cu) (net 6))
@@
   (segment (start 144.8 86.775) (end 144.8 86) (width 0.4) (layer F.Cu) (net 6))
   (segment (start 147.592102 76.592102) (end 146 75) (width 0.8) (layer F.Cu) (net 6))
-  (segment (start 146 68) (end 146 75) (width 0.8) (layer F.Cu) (net 6))
-  (segment (start 150 64) (end 160.87931 64) (width 0.8) (layer F.Cu) (net 6))
-  (segment (start 150 64) (end 146 68) (width 0.8) (layer F.Cu) (net 6))
+  (segment (start 146 72.75) (end 146 75) (width 0.8) (layer F.Cu) (net 6))
+  (segment (start 155.5 64) (end 160.87931 64) (width 0.8) (layer F.Cu) (net 6))
   (segment (start 147.592102 76.592102) (end 147.592102 77.407898) (width 0.8) (layer F.Cu) (net 6))
   (segment (start 160.882133 63.997177) (end 160.87931 64) (width 0.8) (layer F.Cu) (net 6))
