File: hardware/BlackWolf_1.0/micromouse.kicad_pcb (KiCad board)
At the start: 2 copper layers, 100 x 74 mm, 79 parts, among them CN1 5_PIN_HEADER, CN2 5_PIN_HEADER, J1 uSD_SLOT_47219-2001, M1 MOTOR_MOUNTS_AND_ENCODERS, M3 2.54MM-SLIDE-SWITCH_TS02_SWIT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, P1 B3B-PH-SM4-TB, P2 B3B-PH-SM4-TB, SW1 SWITCH_DPST, SW2 SWITCH_DPST, SW3 SWITCH_DPST, U1 STM32F446RE_LQFP64, U10 MPU-9250, U11 TPS76850, U12 TPS73633, U2 MAX14871, U3 MAX14871, U4 TCA9545A, U5 VL6180X_POLOLU, U6 VL6180X_POLOLU, U7 VL6180X_POLOLU, U8 VL6180X_POLOLU, U9 HCMS-2901

Commit message: added BlackWolf hardware project - on progress!
Parts:
- removed C_RANGE1: 0.1uF, footprints_micromouse:C_0603
- removed C_uSD1: 10uF, footprints_micromouse:C_1206
- removed D1: Led_Small, footprints_micromouse:LED_0603
- removed J1: uSD_SLOT_47219-2001, footprints_micromouse:uSD_MOLEX_47219-2001
- removed R_RANGE1, R_RANGE2, R_RANGE3, R_RANGE4, R_RANGE5, R_RANGE6, R_RANGE7: 10k, footprints_micromouse:R_0603
- removed R_uSD1: 1k, footprints_micromouse:R_0603
- removed U4: TCA9545A, footprints_micromouse:TSSOP-20_4.4x6.5mm_Pitch0.65mm
- removed U5, U6, U7, U8: VL6180X_POLOLU, footprints_micromouse:VL6180X_POLOLU_Pin_Header_Straight_1x07
- added C_F1: 4.7u, footprints_micromouse:C_0603, F.Cu at (155.0, 120.8)
- added C_F2: 0.1u, footprints_micromouse:C_0603, F.Cu at (156.6, 120.2)
- added C_F3: 4.7u, footprints_micromouse:C_0603, F.Cu at (149.8, 100.2)
- added C_F4: 0.1u, footprints_micromouse:C_0603, F.Cu at (151.5, 100.2)
- added C_F5: 4.7u, footprints_micromouse:C_0603, F.Cu at (149.2, 78.0)
- added C_F6: 0.1u, footprints_micromouse:C_0603, F.Cu at (151.0, 80.5)
- added C_F7: 4.7u, footprints_micromouse:C_0603, F.Cu at (156.5, 69.2)
- added C_F8: 0.1u, footprints_micromouse:C_0603, F.Cu at (156.5, 70.9)
- added C_PB1: 0.1uF, footprints_micromouse:C_0603, F.Cu at (221.0, 114.0)
- added C_PB2: 0.1uF, footprints_micromouse:C_0603, F.Cu at (228.5, 114.0)
- added D_F1: SFH 4545, Pin_Headers:Pin_Header_Straight_1x02_Pitch2.54mm, F.Cu at (155.5, 113.5)
- added D_F2: SFH 4545, Pin_Headers:Pin_Header_Straight_1x02_Pitch2.54mm, F.Cu at (148.2, 96.8)
- added D_F3: SFH 4545, Pin_Headers:Pin_Header_Straight_1x02_Pitch2.54mm, F.Cu at (146.2, 84.2)
- added D_F4: SFH 4545, Pin_Headers:Pin_Header_Straight_1x02_Pitch2.54mm, F.Cu at (156.0, 64.0)
- added LED_BLUE2: Led_Small, footprints_micromouse:LED_0603, F.Cu at (179.8, 110.0)
- added LED_RED2: Led_Small, footprints_micromouse:LED_0603, F.Cu at (179.8, 108.2)
- added LEFT: RANGE_SENSOR_HOUSING, footprints_micromouse:RANGE_SENSOR_HOUSING, F.Cu at (143.0, 99.5)
- added LEFT_FRONT: RANGE_SENSOR_HOUSING, footprints_micromouse:RANGE_SENSOR_HOUSING, F.Cu at (150.0, 116.0)
- added M2: LEFT_MOTOR, Pin_Headers:Pin_Header_Straight_1x02_Pitch2.00mm, F.Cu at (232.4, 92.1)
- added M4: RIGHT_MOTOR, Pin_Headers:Pin_Header_Straight_1x02_Pitch2.00mm, F.Cu at (232.4, 88.3)
- added Q1: DMN3150LW, TO_SOT_Packages_SMD:SOT-323_SC-70, F.Cu at (160.5, 120.2)
- added Q2: DMN3150LW, TO_SOT_Packages_SMD:SOT-323_SC-70, F.Cu at (155.5, 100.0)
- added Q3: DMN3150LW, TO_SOT_Packages_SMD:SOT-323_SC-70, F.Cu at (153.2, 81.2)
- added Q4: DMN3150LW, TO_SOT_Packages_SMD:SOT-323_SC-70, F.Cu at (158.8, 59.1)
- added Q5: TEFT4300, Pin_Headers:Pin_Header_Straight_1x02_Pitch2.54mm, F.Cu at (152.5, 114.0)
- added Q6: TEFT4300, Pin_Headers:Pin_Header_Straight_1x02_Pitch2.54mm, F.Cu at (144.5, 97.0)
- added Q7: TEFT4300, Pin_Headers:Pin_Header_Straight_1x02_Pitch2.54mm, F.Cu at (144.2, 82.2)
- added Q8: TEFT4300, Pin_Headers:Pin_Header_Straight_1x02_Pitch2.54mm, F.Cu at (153.0, 63.5)
- added R5: 1k, footprints_micromouse:R_0603, F.Cu at (182.6, 108.2)
- added R6: 1k, footprints_micromouse:R_0603, F.Cu at (182.6, 110.0)
- added RIGHT: RANGE_SENSOR_HOUSING, footprints_micromouse:RANGE_SENSOR_HOUSING, F.Cu at (143.0, 79.5)
- added RIGHT_FRONT: RANGE_SENSOR_HOUSING, footprints_micromouse:RANGE_SENSOR_HOUSING, F.Cu at (150.0, 64.0)
- added R_F1: 47k, footprints_micromouse:R_0603, F.Cu at (158.2, 120.0)
- added R_F10: 2.4k, footprints_micromouse:R_0603, F.Cu at (147.0, 103.2)
- added R_F11: 2.4k, footprints_micromouse:R_0603, F.Cu at (145.8, 74.5)
- added R_F12: 2.4k, footprints_micromouse:R_0603, F.Cu at (153.3, 58.9)
- added R_F2: 10, footprints_micromouse:R_0603, F.Cu at (160.5, 117.5)
- added R_F3: 47k, footprints_micromouse:R_0603, F.Cu at (153.2, 100.0)
- added R_F4: 10, footprints_micromouse:R_0603, F.Cu at (154.0, 96.0)
- added R_F5: 47k, footprints_micromouse:R_0603, F.Cu at (155.5, 81.5)
- added R_F6: 10, footprints_micromouse:R_0603, F.Cu at (151.8, 84.5)
- added R_F7: 47k, footprints_micromouse:R_0603, F.Cu at (161.1, 59.1)
- added R_F8: 10, footprints_micromouse:R_0603, F.Cu at (159.2, 62.3)
- added R_F9: 2.4k, footprints_micromouse:R_0603, F.Cu at (152.5, 121.0)
- CN1: value 5_PIN_HEADER -> 7_PIN_HEADER; footprint footprints_micromouse:Pin_Header_Straight_1x05 -> Pin_Headers:Pin_Header_Straight_1x07_Pitch2.54mm
- CN2: footprint footprints_micromouse:Pin_Header_Straight_1x05 -> Pin_Headers:Pin_Header_Straight_1x06_Pitch2.54mm
- C_VCAP1: value 2.2uF -> 4.7uF
- R_PB1, R_PB2: value 47k -> 1k
- moved M3 64.9 mm to (224.8, 57.1)
- moved SW1 61.0 mm to (223.0, 120.0)
- moved SW2 59.3 mm to (230.5, 120.0), turned to 90 degrees
- moved P2 54.8 mm to (229.9, 62.2)
- moved R_PB2 48.8 mm to (231.5, 114.0)
- moved R_PB1 48.6 mm to (224.0, 114.0)
- moved P1 43.7 mm to (229.9, 67.3)
- moved C_IMU3 39.4 mm to (142.4, 90.0)
- moved SW3 39.1 mm to (162.4, 70.0), turned to 90 degrees
- moved C_IMU2 36.5 mm to (144.3, 90.0)
- moved C_IMU1 35.9 mm to (146.1, 90.1), turned to 90 degrees
- moved C_RESET1 35.2 mm to (163.6, 75.9), turned to 0 degrees
- moved L_BEAD1 32.5 mm to (154.0, 56.5), turned to 180 degrees
- moved U10 30.9 mm to (149.0, 90.0), turned to 270 degrees
- moved R_IMU2 26.8 mm to (152.0, 88.0), turned to 270 degrees
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Connections:
- C_V6 pad 1: GND -> +3V3
- C_V6 pad 2: +3V3 -> GND
- C_VCAP1 pad 1: Net-(C_VCAP1-Pad1) -> GND
- C_VCAP1 pad 2: GND -> Net-(C_VCAP1-Pad2)
- R_IMU1 pad 2: IMU_SCL -> /uSD_IMU_DISPLAY/IMU_SCL
- R_IMU2 pad 2: IMU_SDA -> /uSD_IMU_DISPLAY/IMU_SDA
- R_PB1 pad 1: PB1 -> Net-(C_PB1-Pad1)
- R_PB2 pad 1: PB2 -> Net-(C_PB2-Pad1)
- R_VOL1 pad 2: VOL_METER -> BATT_LEVEL
- R_VOL2 pad 1: VOL_METER -> BATT_LEVEL
- SW1 pad 2: +3V3 -> GND
- SW2 pad 2: +3V3 -> GND
- U1 pad PA0_: Net-(U1-PadPA0_) -> EMITTER_SIDES
- U1 pad PA1: Net-(U1-PadPA1) -> EMITTER_FL
- U1 pad PA12: PB2 -> Net-(U1-PadPA12)
- U1 pad PA15: PB1 -> Net-(U1-PadPA15)
- U1 pad PA6: Net-(U1-PadPA6) -> BATT_LEVEL
- U1 pad PB10: IMU_SCL -> LED4
- U1 pad PB11: Net-(C_VCAP1-Pad1) -> Net-(C_VCAP1-Pad2)
- U1 pad PB12: ~uSD_SS -> LED5
- U1 pad PB13: uSD_SCK -> LED6
- U1 pad PB14: uSD_MISO -> PB1
- U1 pad PB15: uSD_MOSI -> PB2
- U1 pad PB2: IMU_INT -> LED3
- U1 pad PB4: Net-(U1-PadPB4) -> ROT_R_CHA
- U1 pad PB5: VOL_METER -> ROT_R_CHB
- U1 pad PB6: ROT_R_CHA -> Net-(U1-PadPB6)
- U1 pad PB7: ROT_R_CHB -> IMU_INT
- U1 pad PB8: RANGE_SCL -> IMU_SCL
- U1 pad PB9: RANGE_SDA -> IMU_SDA
- U1 pad PC0: Net-(U1-PadPC0) -> RECV_FR
- U1 pad PC1: Net-(U1-PadPC1) -> RECV_R
- U1 pad PC10: LED4 -> Net-(U1-PadPC10)
- U1 pad PC11: LED3 -> Net-(U1-PadPC11)
- U1 pad PC12: IMU_SDA -> Net-(U1-PadPC12)
- U1 pad PC13: ~RANGE_RESET -> EMITTER_FR
- U1 pad PC2: Net-(U1-PadPC2) -> RECV_L
- U1 pad PC3: Net-(U1-PadPC3) -> RECV_FL
- U10 pad 12: IMU_INT -> /uSD_IMU_DISPLAY/IMU_INT
- U10 pad 23: IMU_SCL -> /uSD_IMU_DISPLAY/IMU_SCL
- U10 pad 24: IMU_SDA -> /uSD_IMU_DISPLAY/IMU_SDA
- U2 pad 14: Net-(M1-PadL_MB) -> Net-(M2-Pad2)
- U2 pad 15: Net-(M1-PadL_MB) -> Net-(M2-Pad2)
- U2 pad 2: Net-(M1-PadL_MA) -> Net-(M2-Pad1)
- U2 pad 3: Net-(M1-PadL_MA) -> Net-(M2-Pad1)
- U3 pad 14: Net-(M1-PadR_MB) -> Net-(M4-Pad2)
- U3 pad 15: Net-(M1-PadR_MB) -> Net-(M4-Pad2)
- U3 pad 2: Net-(M1-PadR_MA) -> Net-(M4-Pad1)
- U3 pad 3: Net-(M1-PadR_MA) -> Net-(M4-Pad1)
Routing:
- net ~uSD_SS: track 94.1 -> 0.00 mm, vias 4 -> 0
- net uSD_SCK: track 86.4 -> 0.00 mm, vias 4 -> 0
- net uSD_MOSI: track 78.5 -> 0.00 mm, vias 4 -> 0
- net +3V3: track 266.0 -> 190.3 mm, vias 8 -> 7
- net uSD_MISO: track 72.6 -> 0.00 mm, vias 4 -> 0
- net +BATT: track 173.9 -> 104.0 mm
- net LED4: track 56.0 -> 12.4 mm, vias 2 -> 0
- net RANGE_SCL: track 43.5 -> 0.00 mm, vias 2 -> 0
- net RECV_FL: track 0.00 -> 42.9 mm, vias 0 -> 2
- net EMITTER_SIDES: track 0.00 -> 42.8 mm
- net RECV_FR: track 0.00 -> 42.7 mm, vias 0 -> 1
- net LED3: track 52.5 -> 10.3 mm, vias 2 -> 0
- net GND: track 508.1 -> 467.4 mm
- net RECV_R: track 0.00 -> 40.5 mm, vias 0 -> 1
- net RESET: track 83.5 -> 43.1 mm, vias 4 -> 1
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- added copper zone on F.Cu, net +3.3VADC

Commit message: BlackWolf PCB design completed
Parts:
- moved R_MOTOR1 20.7 mm to (197.5, 92.4)
- moved R_MOTOR2 13.9 mm to (204.8, 89.4)
- moved R13 13.5 mm to (220.5, 95.5), turned to 270 degrees
- moved R14 13.5 mm to (220.5, 84.5), turned to 90 degrees
- moved M2 12.9 mm to (219.5, 91.5)
- moved C_MOTOR2 12.3 mm to (227.2, 79.8)
- moved C_MOTOR1 12.3 mm to (226.5, 101.0)
- moved M4 10.9 mm to (221.5, 88.5), turned to 270 degrees
- moved U2 10.1 mm to (220.5, 100.7), turned to 0 degrees
- moved U3 10.1 mm to (220.5, 79.3), turned to 180 degrees
- moved C_M1 10.0 mm to (230.0, 90.0), turned to 180 degrees
- moved P1 0.34 mm to (230.0, 67.0), turned to 180 degrees
- moved R_F12 0.30 mm to (153.0, 58.9)
- moved P2 0.26 mm to (230.0, 62.0), turned to 180 degrees
Connections:
- R_IMU1 pad 2: /uSD_IMU_DISPLAY/IMU_SCL -> IMU_SCL
- R_IMU2 pad 2: /uSD_IMU_DISPLAY/IMU_SDA -> IMU_SDA
- U10 pad 12: /uSD_IMU_DISPLAY/IMU_INT -> IMU_INT
- U10 pad 23: /uSD_IMU_DISPLAY/IMU_SCL -> IMU_SCL
- U10 pad 24: /uSD_IMU_DISPLAY/IMU_SDA -> IMU_SDA
Routing:
- net +3V3: track 190.3 -> 286.7 mm, vias 7 -> 12
- net +BATT: track 104.0 -> 139.8 mm, vias 3 -> 0
- net IMU_INT: track 21.0 -> 38.3 mm, vias 2 -> 4
- net /uSD_IMU_DISPLAY/IMU_INT: track 16.6 -> 0.00 mm, vias 2 -> 0
- net (no net): track 9.15 -> 25.6 mm, vias 3 -> 6
- net GND: track 467.4 -> 459.3 mm, vias 37 -> 45
- net IMU_SCL: track 22.9 -> 30.9 mm
- net /uSD_IMU_DISPLAY/IMU_SCL: track 7.34 -> 0.00 mm
- net IMU_SDA: track 22.3 -> 29.6 mm
- net /uSD_IMU_DISPLAY/IMU_SDA: track 7.10 -> 0.00 mm
- net Net-(M2-Pad1): track 20.1 -> 13.1 mm
- net ~MOTOR_R_FAULT: track 43.1 -> 38.0 mm
- net MOTOR_R_PWM: track 55.6 -> 50.5 mm, vias 2 -> 0
- net Net-(R13-Pad1): track 23.4 -> 28.2 mm
- net Net-(M4-Pad1): track 17.9 -> 13.2 mm
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
Commit message: Changed Slikscreen
Other:
- board text added: "BlackWolf v1.0"
- board text removed: "WolfieMouse"
Changed lines of the file:
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@@
     (links 256)
     (no_connects 0)
-    (area 136.924999 52.924999 237.075001 127.075001)
+    (area -79.564284 -59.170945 338.85 238.170945)
     (thickness 1.6)
     (drawings 42)
@@
   )
   (setup
-    (last_trace_width 0.4)
+    (last_trace_width 0.25)
     (user_trace_width 0.2)
     (user_trace_width 0.28)
@@
     (tags "resistor 1206")
     (attr smd)
-    (fp_text reference R14 (at -3 1 90) (layer F.SilkS)
+    (fp_text reference R14 (at -0.082 1.75 90) (layer F.SilkS)
       (effects (font (size 0.5 0.5) (thickness 0.1)))
     )
@@
     (tags "resistor 1206")
     (attr smd)
-    (fp_text reference R13 (at -3 -1 270) (layer F.SilkS)
+    (fp_text reference R13 (at 0.004 -1.75 270) (layer F.SilkS)
       (effects (font (size 0.5 0.5) (thickness 0.1)))
     )
@@
     (tags "capacitor 1206")
     (attr smd)
-    (fp_text reference C_VCAP2 (at 0.75 -1.75 270) (layer F.SilkS)
+    (fp_text reference C_VCAP2 (at 2.86 -1.48 270) (layer F.SilkS)
       (effects (font (size 0.5 0.5) (thickness 0.1)))
     )
@@
     (tags "capacitor 1206")
     (attr smd)
-    (fp_text reference C_3.3V1 (at -1 -1.5) (layer F.SilkS)
+    (fp_text reference C_3.3V1 (at -2.382 -1.538) (layer F.SilkS)
       (effects (font (size 0.5 0.5) (thickness 0.1)))
     )
@@
     (tags "resistor 0603")
     (attr smd)
-    (fp_text reference R_MOTOR2 (at 3.25 0 90) (layer F.SilkS)
+    (fp_text reference R_MOTOR2 (at 1.77 1.448 90) (layer F.SilkS)
       (effects (font (size 0.5 0.5) (thickness 0.1)))
     )
@@
     (tags "resistor 0603")
     (attr smd)
-    (fp_text reference R_MOTOR1 (at -3.25 0 90) (layer F.SilkS)
+    (fp_text reference R_MOTOR1 (at -0.056 -1.412 90) (layer F.SilkS)
       (effects (font (size 0.5 0.5) (thickness 0.1)))
     )
@@
     (tags "LED led 0603 SMD smd SMT smt smdled SMDLED smtled SMTLED")
     (attr smd)
-    (fp_text reference D_PWR1 (at 2.85 -0.4 90) (layer F.SilkS)
+    (fp_text reference D_PWR1 (at 1.846 -1.156 90) (layer F.SilkS)
       (effects (font (size 0.5 0.5) (thickness 0.1)))
     )
@@
       (effects (font (size 0.8 0.8) (thickness 0.05)))
     )
-    (fp_text value MPU-9250 (at 0 8 270) (layer F.SilkS)
+    (fp_text value MPU-9250 (at 0 9 270) (layer F.SilkS)
       (effects (font (size 1 0.9) (thickness 0.05)))
     )
@@
     (tags "capacitor 0603")
     (attr smd)
-    (fp_text reference C_IMU1 (at 3 0.1 90) (layer F.SilkS)
+    (fp_text reference C_IMU1 (at 2.5 0.3 180) (layer F.SilkS)
       (effects (font (size 0.5 0.5) (thickness 0.1)))
     )
@@
     (tags "capacitor 0603")
     (attr smd)
-    (fp_text reference C_IMU3 (at 3 -0.05 90) (layer F.SilkS)
+    (fp_text reference C_IMU3 (at 0 -1.15 90) (layer F.SilkS)
       (effects (font (size 0.5 0.5) (thickness 0.1)))
     )
@@
     (tags "capacitor 0603")
     (attr smd)
-    (fp_text reference C_RESET1 (at 0 -1.25) (layer F.SilkS)
+    (fp_text reference C_RESET1 (at 0 1.24) (layer F.SilkS)
       (effects (font (size 0.5 0.5) (thickness 0.1)))
     )
@@
     (tags "capacitor 0603")
     (attr smd)
-    (fp_text reference C_V4 (at 0 -1.25) (layer F.SilkS)
+    (fp_text reference C_V4 (at -0.794 1.36) (layer F.SilkS)
       (effects (font (size 0.5 0.5) (thickness 0.1)))
     )
@@
     (tags "capacitor 0603")
     (attr smd)
-    (fp_text reference C_V6 (at -2.5 0 90) (layer F.SilkS)
+    (fp_text reference C_V6 (at -0.254 -1.016 90) (layer F.SilkS)
       (effects (font (size 0.5 0.5) (thickness 0.1)))
     )
@@
       (effects (font (size 0.75 0.75) (thickness 0.05)))
     )
-    (fp_text value MAX14871 (at 0 -2.25 180) (layer F.SilkS)
+    (fp_text value MAX14871 (at -0.226 3.1 180) (layer F.SilkS)
       (effects (font (size 0.5 0.5) (thickness 0.1)))
     )
@@
     (tags "capacitor 0805")
     (attr smd)
-    (fp_text reference C_IMU2 (at 2.4 0.1 180) (layer F.SilkS)
+    (fp_text reference C_IMU2 (at 2.25 -0.8 180) (layer F.SilkS)
       (effects (font (size 0.5 0.5) (thickness 0.1)))
     )
@@
     (tags "capacitor 1210")
     (attr smd)
-    (fp_text reference C_VBAT1 (at 3.05 1.15 90) (layer F.SilkS)
+    (fp_text reference C_VBAT1 (at 2.696 2.632 90) (layer F.SilkS)
       (effects (font (size 0.75 0.75) (thickness 0.1)))
     )
@@
     (descr "Through hole straight pin header, 1x02, 2.54mm pitch, single row")
     (tags "Through hole pin header THT 1x02 2.54mm single row")
-    (fp_text reference D_F3 (at 2.298097 1.59099 225) (layer F.SilkS)
+    (fp_text reference D_F3 (at -2.262742 1.343503 405) (layer F.SilkS)
       (effects (font (size 1 1) (thickness 0.15)))
     )
@@
       (effects (font (size 1 1) (thickness 0.15)))
     )
-    (fp_text value "SFH 4545" (at 0 4.87 350) (layer F.Fab)
+    (fp_text value "SFH 4545" (at 2.560662 2.543995 620) (layer F.Fab) hide
       (effects (font (size 1 1) (thickness 0.15)))
     )
@@
     (fp_line (start 1.8 4.35) (end 1.8 -1.8) (layer F.CrtYd) (width 0.05))
     (fp_line (start 1.8 -1.8) (end -1.8 -1.8) (layer F.CrtYd) (width 0.05))
-    (fp_text user %R (at 0 -2.33 350) (layer F.Fab)
+    (fp_text user %R (at -0.104934 4.760545 350) (layer F.Fab) hide
       (effects (font (size 1 1) (thickness 0.15)))
     )
@@
     (descr "Through hole straight pin header, 1x02, 2.54mm pitch, single row")
     (tags "Through hole pin header THT 1x02 2.54mm single row")
-    (fp_text reference Q7 (at -0.353553 5.868986 135) (layer F.SilkS)
+    (fp_text reference Q7 (at 0.670337 5.371183 135) (layer F.SilkS)
       (effects (font (size 1 1) (thickness 0.15)))
     )
@@
     (descr "Through hole straight pin header, 1x02, 2.54mm pitch, single row")
     (tags "Through hole pin header THT 1x02 2.54mm single row")
-    (fp_text reference Q8 (at 0 -2.33 350) (layer F.SilkS)
+    (fp_text reference Q8 (at -0.480102 5.339488 350) (layer F.SilkS)
       (effects (font (size 1 1) (thickness 0.15)))
     )
-    (fp_text value TEFT4300 (at 0 4.87 350) (layer F.Fab)
+    (fp_text value TEFT4300 (at -2.341953 1.40299 440) (layer F.Fab) hide
       (effects (font (size 1 1) (thickness 0.15)))
     )
@@
     (fp_line (start 1.8 4.35) (end 1.8 -1.8) (layer F.CrtYd) (width 0.05))
     (fp_line (start 1.8 -1.8) (end -1.8 -1.8) (layer F.CrtYd) (width 0.05))
-    (fp_text user %R (at 0 -2.33 350) (layer F.Fab)
+    (fp_text user %R (at -3.771591 3.228986 440) (layer F.Fab) hide
       (effects (font (size 1 1) (thickness 0.15)))
     )
@@
     (tags "resistor 0603")
     (attr smd)
-    (fp_text reference R_F12 (at 0 -1.2 90) (layer F.SilkS)
+    (fp_text reference R_F12 (at -0.028 1.178 90) (layer F.SilkS)
       (effects (font (size 0.5 0.5) (thickness 0.1)))
     )
@@
     (tags "resistor 0603")
     (attr smd)
-    (fp_text reference R_F10 (at 2.5 0) (layer F.SilkS)
+    (fp_text reference R_F10 (at -0.25 1.5) (layer F.SilkS)
       (effects (font (size 0.5 0.5) (thickness 0.1)))
     )
@@
     (tags "resistor 0603")
     (attr smd)
-    (fp_text reference R_F8 (at -2.3 0.1 90) (layer F.SilkS)
+    (fp_text reference R_F8 (at -0.11 1.28 90) (layer F.SilkS)
       (effects (font (size 0.5 0.5) (thickness 0.1)))
     )
@@
     (tags "resistor 0603")
     (attr smd)
-    (fp_text reference R_F7 (at 0 -1.2 90) (layer F.SilkS)
+    (fp_text reference R_F7 (at 2.204 0.698 90) (layer F.SilkS)
       (effects (font (size 0.5 0.5) (thickness 0.1)))
     )
@@
     (tags "capacitor 0603")
     (attr smd)
-    (fp_text reference C_F8 (at 0 -1.25) (layer F.SilkS)
+    (fp_text reference C_F8 (at -2.4 0.15) (layer F.SilkS)
       (effects (font (size 0.5 0.5) (thickness 0.1)))
     )
@@
     (tags "capacitor 0603")
     (attr smd)
-    (fp_text reference C_F7 (at 0 -1.25) (layer F.SilkS)
+    (fp_text reference C_F7 (at -2.45 0.35) (layer F.SilkS)
       (effects (font (size 0.5 0.5) (thickness 0.1)))
     )
@@
     (tags "LED led 0603 SMD smd SMT smt smdled SMDLED smtled SMTLED")
     (attr smd)
-    (fp_text reference LED_RED2 (at -1 -1.1) (layer F.SilkS)
+    (fp_text reference LED_RED2 (at 5.918 -0.204) (layer F.SilkS)
       (effects (font (size 0.5 0.5) (thickness 0.1)))
     )
@@
     (tags "LED led 0603 SMD smd SMT smt smdled SMDLED smtled SMTLED")
     (attr smd)
-    (fp_text reference LED_BLUE2 (at -1 -1.1) (layer F.SilkS)
+    (fp_text reference LED_BLUE2 (at 2.168 1.268) (layer F.SilkS)
       (effects (font (size 0.5 0.5) (thickness 0.1)))
     )
@@
     (tags "resistor 0603")
     (attr smd)
-    (fp_text reference R5 (at 0 -1.2 180) (layer F.SilkS)
+    (fp_text reference R5 (at -1.874 -0.546 180) (layer F.SilkS)
       (effects (font (size 0.5 0.5) (thickness 0.1)))
     )
@@
     (tags "resistor 0603")
     (attr smd)
-    (fp_text reference R6 (at 0 -1.2 180) (layer F.SilkS)
+    (fp_text reference R6 (at -1.874 -0.518 180) (layer F.SilkS)
       (effects (font (size 0.5 0.5) (thickness 0.1)))
     )
@@
     (arrow2b (pts (xy 255 53) (xy 255.586421 54.126504)))
   )
-  (gr_text WolfieMouse (at 240.665 94.615 90) (layer F.SilkS)
+  (gr_text "BlackWolf v1.0" (at 233 92.25 90) (layer F.SilkS)
     (effects (font (size 2.5 2.5) (thickness 0.3)))
   )
-  (gr_text "Designed by:\nBumsik Kim" (at 245.11 97.155 90) (layer F.SilkS)
+  (gr_text "Designed by:\nBumsik Kim" (at 226.568 109.22) (layer F.SilkS)
     (effects (font (size 1.8 1.8) (thickness 0.3)))
   )
