File: hardware/BlackWolf_1.0/micromouse.sch (KiCad schematic (older format))
At the start: 44 parts, among them CN1 5_PIN_HEADER, CN2 5_PIN_HEADER, M3 2.54MM-SLIDE-SWITCH_TS02_SWIT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, P1 B3B-PH-SM4-TB, P2 B3B-PH-SM4-TB, SW1 SWITCH_DPST, SW2 SWITCH_DPST, SW3 SWITCH_DPST, U1 STM32F446RE_LQFP64, U11 TPS76850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

Commit message: added BlackWolf hardware project - on progress!
Parts:
- removed CN1: 5_PIN_HEADER, Pin_Headers:Pin_Header_Straight_1x05, symbol 5_PIN_HEADER
- added CN1: 7_PIN_HEADER, Pin_Headers:Pin_Header_Straight_1x07_Pitch2.54mm, symbol 7_PIN_HEADER
- added C_PB1, C_PB2: 0.1uF, Capacitors_SMD:C_0603, symbol C_Small
- added LED_BLUE2, LED_RED2: Led_Small, LEDs:LED_0603, symbol Led_Small
- added R5, R6: 1k, Resistors_SMD:R_0603, symbol R_Small
- CN2: footprint Pin_Headers:Pin_Header_Straight_1x05 -> Pin_Headers:Pin_Header_Straight_1x06_Pitch2.54mm; symbol 5_PIN_HEADER -> 6_PIN_HEADER
- C_VCAP1: value 2.2uF -> 4.7uF; footprint Capacitors_SMD:C_1206 -> Capacitors_SMD:C_0603
- R_PB1, R_PB2: value 47k -> 1k
Connections:
- net labels added: BATT_LEVEL, EMITTER_FL, EMITTER_FR, EMITTER_SIDES, LED5, LED6, RECV_FL, RECV_FR, RECV_L, RECV_R
- net labels removed: RANGE_SCL, RANGE_SDA, VOL_METER, ~RANGE_RESET
- wire segments 256 -> 233
- no-connect marks 0 -> 4
Other:
- note added: "Both PB1 and PB2\nshoul be internally\npulled-up"
- note added: "uSD & IMU\n& DISPLAY"
- note removed: "uSD & IMU & DISPLAY"
- moved on the sheet: CNR1, C_3.3V1, C_3.3V2, C_5V1, C_5V2, C_M1, C_RESET1, C_V1, C_V2, C_V3, C_V4, C_V5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

Commit message: BlackWolf PCB design completed
Connections:
- net labels removed: uSD_MISO, uSD_MOSI, uSD_SCK, ~uSD_SS
- wire segments 233 -> 234
- no-connect marks 4 -> 25
Changed lines of the file:
@@
 Text GLabel 2950 6600 3    40   Input ~ 0
 DIS_SCK
-Text GLabel 9600 2950 0    40   Input ~ 0
-~uSD_SS
-Text GLabel 9600 3050 0    40   Input ~ 0
-uSD_SCK
-Text GLabel 9600 3250 0    40   Input ~ 0
-uSD_MISO
-Text GLabel 9600 3150 0    40   Input ~ 0
-uSD_MOSI
 Text GLabel 9600 3550 0    40   Input ~ 0
 ~DIS_CE
@@
 Wire Wire Line
 	9650 5450 9650 5800
+Text GLabel 9600 4100 0    40   Input ~ 0
+IMU_SDA
+Text GLabel 9600 4000 0    40   Input ~ 0
+IMU_SCL
+Text GLabel 9600 4200 0    40   Input ~ 0
+IMU_INT
+NoConn ~ 4100 1650
+NoConn ~ 3600 2000
+NoConn ~ 3600 1450
+NoConn ~ 5300 1400
+NoConn ~ 5300 1450
+NoConn ~ 9100 1350
+NoConn ~ 9100 1450
+NoConn ~ 9100 1750
+NoConn ~ 10100 1750
+Wire Wire Line
+	3450 3550 3450 3400
+NoConn ~ 3950 3400
+NoConn ~ 3850 3400
+NoConn ~ 3750 3400
+NoConn ~ 3650 3400
+NoConn ~ 3550 3400
+NoConn ~ 3450 3400
+NoConn ~ 3150 3400
+NoConn ~ 4900 4550
+NoConn ~ 9600 2950
+NoConn ~ 9600 3050
+NoConn ~ 9600 3150
+NoConn ~ 9600 3250
 $EndSCHEMATC
