File: hardware/BlackWolf_1.0/motor.sch (KiCad schematic (older format))
At the start: 9 parts, among them M1 MOTOR_MOUNTS_AND_ENCODERS, U2 MAX14871, U3 MAX14871

Commit message: added BlackWolf hardware project - on progress!
Parts:
- added M2: LEFT_MOTOR, Pin_Headers:Pin_Header_Straight_1x02_Pitch2.00mm, symbol MOTOR
- added M4: RIGHT_MOTOR, Pin_Headers:Pin_Header_Straight_1x02_Pitch2.00mm, symbol MOTOR
Changed lines of the file:
@@
 	1    0    0    -1
-$EndComp
-$Comp
-L MOTOR_MOUNTS_AND_ENCODERS M1
-U 1 1 56EB6456
-P 7450 3900
-F 0 "M1" H 6550 4600 45  0001 C CNN
-F 1 "MOTOR_MOUNTS_AND_ENCODERS" H 7400 4350 50  0000 C CNN
-F 2 "footprints_micromouse:FUTURA-1.0-MOTOR-MOUNT-TEMPLATE" H 8100 4600 20  0001 C CNN
-F 3 "" H 7450 3850 60  0000 C CNN
-	1    7450 3900
-	0    1    1    0
 $EndComp
 Wire Wire Line
@@
 Connection ~ 5000 5050
 $Comp
-L GND #PWR035
+L GND #PWR033
 U 1 1 56EB8B5A
 P 6700 4650
-F 0 "#PWR035" H 6700 4400 50  0001 C CNN
+F 0 "#PWR033" H 6700 4400 50  0001 C CNN
 F 1 "GND" H 6700 4500 50  0000 C CNN
 F 2 "" H 6700 4650 50  0000 C CNN
@@
 ~R_FAULT
 $Comp
-L +BATT #PWR036
+L +BATT #PWR034
 U 1 1 56EB8FD2
 P 4250 2000
-F 0 "#PWR036" H 4250 1850 50  0001 C CNN
+F 0 "#PWR034" H 4250 1850 50  0001 C CNN
 F 1 "+BATT" H 4250 2140 50  0000 C CNN
 F 2 "" H 4250 2000 50  0000 C CNN
@@
 $EndComp
 $Comp
-L +5V #PWR037
+L +5V #PWR035
 U 1 1 56EC1082
 P 6600 3200
-F 0 "#PWR037" H 6600 3050 50  0001 C CNN
+F 0 "#PWR035" H 6600 3050 50  0001 C CNN
 F 1 "+5V" H 6600 3340 50  0000 C CNN
 F 2 "" H 6600 3200 50  0000 C CNN
@@
 	4250 2000 4250 2350
 $Comp
-L +BATT #PWR038
+L +BATT #PWR036
 U 1 1 56ED705F
 P 4250 4150
-F 0 "#PWR038" H 4250 4000 50  0001 C CNN
+F 0 "#PWR036" H 4250 4000 50  0001 C CNN
 F 1 "+BATT" H 4250 4290 50  0000 C CNN
 F 2 "" H 4250 4150 50  0000 C CNN
@@
 	3600 4700 3600 5000
 $Comp
-L GND #PWR039
+L GND #PWR037
 U 1 1 56ED82CD
 P 3550 3400
-F 0 "#PWR039" H 3550 3150 50  0001 C CNN
+F 0 "#PWR037" H 3550 3150 50  0001 C CNN
 F 1 "GND" H 3550 3250 50  0000 C CNN
 F 2 "" H 3550 3400 50  0000 C CNN
@@
 	3550 2950 3550 3400
 $Comp
-L +3.3V #PWR040
+L +3.3V #PWR038
 U 1 1 56ED83FC
 P 3150 3350
-F 0 "#PWR040" H 3150 3200 50  0001 C CNN
+F 0 "#PWR038" H 3150 3200 50  0001 C CNN
 F 1 "+3.3V" H 3150 3490 50  0000 C CNN
 F 2 "" H 3150 3350 50  0000 C CNN
@@
 Connection ~ 4300 5850
 $Comp
-L GND #PWR041
+L GND #PWR039
 U 1 1 56ED9574
 P 3550 5550
-F 0 "#PWR041" H 3550 5300 50  0001 C CNN
+F 0 "#PWR039" H 3550 5300 50  0001 C CNN
 F 1 "GND" H 3550 5400 50  0000 C CNN
 F 2 "" H 3550 5550 50  0000 C CNN
@@
 	3550 5100 3550 5550
 $Comp
-L +3.3V #PWR042
+L +3.3V #PWR040
 U 1 1 56ED957C
 P 3150 5500
-F 0 "#PWR042" H 3150 5350 50  0001 C CNN
+F 0 "#PWR040" H 3150 5350 50  0001 C CNN
 F 1 "+3.3V" H 3150 5640 50  0000 C CNN
 F 2 "" H 3150 5500 50  0000 C CNN
@@
 Connection ~ 3550 5450
 $Comp
-L GNDM #PWR043
+L GNDM #PWR041
 U 1 1 56FA27B2
 P 4300 3750
-F 0 "#PWR043" H 4300 3500 50  0001 C CNN
+F 0 "#PWR041" H 4300 3500 50  0001 C CNN
 F 1 "GNDM" H 4300 3600 50  0000 C CNN
 F 2 "" H 4300 3750 50  0000 C CNN
@@
 $EndComp
 $Comp
-L GNDM #PWR044
+L GNDM #PWR042
 U 1 1 56FA283F
 P 4300 5950
-F 0 "#PWR044" H 4300 5700 50  0001 C CNN
+F 0 "#PWR042" H 4300 5700 50  0001 C CNN
 F 1 "GNDM" H 4300 5800 50  0000 C CNN
 F 2 "" H 4300 5950 50  0000 C CNN
@@
 $EndComp
 $Comp
-L GNDM #PWR045
+L GNDM #PWR043
 U 1 1 57019AE9
 P 4800 4500
-F 0 "#PWR045" H 4800 4250 50  0001 C CNN
+F 0 "#PWR043" H 4800 4250 50  0001 C CNN
 F 1 "GNDM" H 4800 4350 50  0000 C CNN
 F 2 "" H 4800 4500 50  0000 C CNN
@@
 $EndComp
 $Comp
-L GNDM #PWR046
+L GNDM #PWR044
 U 1 1 57019B14
 P 4800 2350
-F 0 "#PWR046" H 4800 2100 50  0001 C CNN
+F 0 "#PWR044" H 4800 2100 50  0001 C CNN
 F 1 "GNDM" H 4800 2200 50  0000 C CNN
 F 2 "" H 4800 2350 50  0000 C CNN
@@
 	4250 4400 4450 4400
 $Comp
-L +3.3V #PWR047
+L +3.3V #PWR045
 U 1 1 5702029E
 P 3600 4300
-F 0 "#PWR047" H 3600 4150 50  0001 C CNN
+F 0 "#PWR045" H 3600 4150 50  0001 C CNN
 F 1 "+3.3V" H 3600 4440 50  0000 C CNN
 F 2 "" H 3600 4300 50  0000 C CNN
@@
 	4250 2250 4450 2250
 $Comp
-L +3.3V #PWR048
+L +3.3V #PWR046
 U 1 1 57020422
 P 3550 2100
-F 0 "#PWR048" H 3550 1950 50  0001 C CNN
+F 0 "#PWR046" H 3550 1950 50  0001 C CNN
 F 1 "+3.3V" H 3550 2240 50  0000 C CNN
 F 2 "" H 3550 2100 50  0000 C CNN
@@
 	1    0    0    -1
 $EndComp
+$Comp
+L MOTOR M2
+U 1 1 58DADD61
+P 7300 2850
+F 0 "M2" H 6400 3550 45  0001 C CNN
+F 1 "LEFT_MOTOR" V 7100 2850 50  0000 C CNN
+F 2 "Pin_Headers:Pin_Header_Straight_1x02_Pitch2.00mm" H 7950 3550 20  0001 C CNN
+F 3 "" H 7200 2800 60  0000 C CNN
+	1    7300 2850
+	0    1    1    0
+$EndComp
+$Comp
+L MOTOR M4
+U 1 1 58DADDFC
+P 7300 4950
+F 0 "M4" H 6400 5650 45  0001 C CNN
+F 1 "RIGHT_MOTOR" V 7500 5000 50  0000 C CNN
+F 2 "Pin_Headers:Pin_Header_Straight_1x02_Pitch2.00mm" H 7950 5650 20  0001 C CNN
+F 3 "" H 7200 4900 60  0000 C CNN
+	1    7300 4950
+	0    1    1    0
+$EndComp
+$Comp
+L MOTOR_MOUNTS_AND_ENCODERS M1
+U 1 1 56EB6456
+P 7450 3900
+F 0 "M1" H 6550 4600 45  0001 C CNN
+F 1 "MOTOR_MOUNTS_AND_ENCODERS" H 7400 4350 50  0000 C CNN
+F 2 "footprints_micromouse:FUTURA-1.0-MOTOR-MOUNT-TEMPLATE" H 8100 4600 20  0001 C CNN
+F 3 "" H 7450 3850 60  0000 C CNN
+	1    7450 3900
+	0    1    1    0
+$EndComp
 $EndSCHEMATC
