File: hardware/BlackWolf_1.0/uSD_IMU_DIS.sch (KiCad schematic (older format))
At the start: 13 parts, among them J1 uSD_SLOT_47219-2001, U10 MPU-9250, U9 HCMS-2901

Commit message: added BlackWolf hardware project - on progress!
Parts:
- removed C_uSD1: 10uF, Capacitors_SMD:C_1206, symbol C_Small
- removed D1: Led_Small, LEDs:LED_0603, symbol Led_Small
- removed J1: uSD_SLOT_47219-2001, footprints_micromouse:uSD_MOLEX_47219-2001, symbol uSD_SLOT_47219-2001
- removed R_uSD1: 1k, Resistors_SMD:R_0603, symbol R_Small
Other:
- note added: "uSD card slot has been removed.\n"
Changed lines of the file:
@@
 	1    0    0    -1
 $EndComp
-$Comp
-L uSD_SLOT_47219-2001 J1
-U 1 1 56EC0AE2
-P 8450 3900
-F 0 "J1" H 7950 4450 50  0000 L CNN
-F 1 "uSD_SLOT_47219-2001" H 7950 4350 50  0000 L CNN
-F 2 "footprints_micromouse:uSD_MOLEX_47219-2001" H 7950 3450 50  0001 L CNN
-F 3 "" H 8450 3900 60  0000 C CNN
-	1    8450 3900
-	1    0    0    -1
-$EndComp
-$Comp
-L +3.3V #PWR060
-U 1 1 56EC0B54
-P 9300 3450
-F 0 "#PWR060" H 9300 3300 50  0001 C CNN
-F 1 "+3.3V" H 9300 3590 50  0000 C CNN
-F 2 "" H 9300 3450 50  0000 C CNN
-F 3 "" H 9300 3450 50  0000 C CNN
-	1    9300 3450
-	1    0    0    -1
-$EndComp
-$Comp
-L GND #PWR061
-U 1 1 56EC0C8A
-P 9300 4250
-F 0 "#PWR061" H 9300 4000 50  0001 C CNN
-F 1 "GND" H 9300 4100 50  0000 C CNN
-F 2 "" H 9300 4250 50  0000 C CNN
-F 3 "" H 9300 4250 50  0000 C CNN
-	1    9300 4250
-	1    0    0    -1
-$EndComp
-Wire Wire Line
-	9150 3600 9550 3600
-Wire Wire Line
-	9300 3600 9300 3450
-Wire Wire Line
-	9150 3800 9300 3800
-Wire Wire Line
-	9300 3800 9300 4250
-Wire Wire Line
-	9150 4200 9550 4200
-Connection ~ 9300 4200
-Wire Wire Line
-	9150 4100 9300 4100
-Connection ~ 9300 4100
-Wire Wire Line
-	9150 4000 9300 4000
-Connection ~ 9300 4000
-Wire Wire Line
-	9150 3900 9300 3900
-Connection ~ 9300 3900
 Text HLabel 7200 4200 0    60   BiDi ~ 0
 ~uSD_SS
@@
 	3800 6200 4450 6200
 $Comp
-L GND #PWR063
+L GND #PWR051
 U 1 1 56EC150D
 P 4100 6550
-F 0 "#PWR063" H 4100 6300 50  0001 C CNN
+F 0 "#PWR051" H 4100 6300 50  0001 C CNN
 F 1 "GND" H 4100 6400 50  0000 C CNN
 F 2 "" H 4100 6550 50  0000 C CNN
@@
 	4450 6200 4450 6150
 $Comp
-L +5V #PWR064
+L +5V #PWR052
 U 1 1 56EC1816
 P 2350 5800
-F 0 "#PWR064" H 2350 5650 50  0001 C CNN
+F 0 "#PWR052" H 2350 5650 50  0001 C CNN
 F 1 "+5V" H 2350 5940 50  0000 C CNN
 F 2 "" H 2350 5800 50  0000 C CNN
@@
 Text Notes 1250 1750 0    200  ~ 40
 MPU_9250 9-DoF IMU Sensor
-Wire Wire Line
-	7200 3600 7750 3600
-Wire Wire Line
-	7200 3800 7750 3800
-Wire Wire Line
-	7200 3900 7750 3900
-Wire Wire Line
-	7200 4200 7750 4200
-$Comp
-L Led_Small D1
-U 1 1 56EC2147
-P 7350 4700
-F 0 "D1" H 7300 4825 50  0000 L CNN
-F 1 "Led_Small" H 7175 4600 50  0001 L CNN
-F 2 "LEDs:LED_0603" V 7350 4700 50  0001 C CNN
-F 3 "" V 7350 4700 50  0000 C CNN
-	1    7350 4700
-	-1   0    0    1
-$EndComp
-$Comp
-L R_Small R_uSD1
-U 1 1 56EC2210
-P 7650 4700
-F 0 "R_uSD1" H 7680 4720 50  0000 L CNN
-F 1 "1k" H 7680 4660 50  0000 L CNN
-F 2 "Resistors_SMD:R_0603" H 7650 4700 50  0001 C CNN
-F 3 "" H 7650 4700 50  0000 C CNN
-	1    7650 4700
-	0    1    1    0
-$EndComp
-Wire Wire Line
-	7300 3600 7300 4500
-Wire Wire Line
-	7300 4500 7200 4500
-Wire Wire Line
-	7200 4500 7200 4700
-Wire Wire Line
-	7200 4700 7250 4700
-Connection ~ 7300 3600
-Wire Wire Line
-	7450 4700 7550 4700
-Wire Wire Line
-	7750 4700 7850 4700
-Wire Wire Line
-	7850 4700 7850 4500
-Wire Wire Line
-	7850 4500 7700 4500
-Wire Wire Line
-	7700 4500 7700 4200
-Connection ~ 7700 4200
-$Comp
-L GND #PWR065
+$Comp
+L GND #PWR053
 U 1 1 56EC2E0A
 P 3450 4050
-F 0 "#PWR065" H 3450 3800 50  0001 C CNN
+F 0 "#PWR053" H 3450 3800 50  0001 C CNN
 F 1 "GND" H 3450 3900 50  0000 C CNN
 F 2 "" H 3450 4050 50  0000 C CNN
@@
 Connection ~ 3450 3900
 $Comp
-L +3.3V #PWR066
+L +3.3V #PWR054
 U 1 1 56EC3332
 P 3500 2100
-F 0 "#PWR066" H 3500 1950 50  0001 C CNN
+F 0 "#PWR054" H 3500 1950 50  0001 C CNN
 F 1 "+3.3V" H 3500 2240 50  0000 C CNN
 F 2 "" H 3500 2100 50  0000 C CNN
@@
 	2300 3150 2300 3200
 $Comp
-L GND #PWR067
+L GND #PWR055
 U 1 1 56EC3E3A
 P 2300 3550
-F 0 "#PWR067" H 2300 3300 50  0001 C CNN
+F 0 "#PWR055" H 2300 3300 50  0001 C CNN
 F 1 "GND" H 2300 3400 50  0000 C CNN
 F 2 "" H 2300 3550 50  0000 C CNN
@@
 	4050 2500 4050 2700
 $Comp
-L GND #PWR068
+L GND #PWR056
 U 1 1 56EC45CA
 P 4050 2700
-F 0 "#PWR068" H 4050 2450 50  0001 C CNN
+F 0 "#PWR056" H 4050 2450 50  0001 C CNN
 F 1 "GND" H 4050 2550 50  0000 C CNN
 F 2 "" H 4050 2700 50  0000 C CNN
@@
 	3900 3400 4100 3400
 $Comp
-L GND #PWR069
+L GND #PWR057
 U 1 1 56EC4DCF
 P 4100 4050
-F 0 "#PWR069" H 4100 3800 50  0001 C CNN
+F 0 "#PWR057" H 4100 3800 50  0001 C CNN
 F 1 "GND" H 4100 3900 50  0000 C CNN
 F 2 "" H 4100 4050 50  0000 C CNN
@@
 $EndComp
 $Comp
-L +3.3V #PWR070
+L +3.3V #PWR058
 U 1 1 56EC6F0F
 P 4650 2500
-F 0 "#PWR070" H 4650 2350 50  0001 C CNN
+F 0 "#PWR058" H 4650 2350 50  0001 C CNN
 F 1 "+3.3V" H 4650 2640 50  0000 C CNN
 F 2 "" H 4650 2500 50  0000 C CNN
@@
 	3400 2650 3400 2200
 $Comp
-L C_Small C_uSD1
-U 1 1 56ED3391
-P 9550 3900
-F 0 "C_uSD1" H 9560 3970 50  0000 L CNN
-F 1 "10uF" H 9570 3820 50  0000 L CNN
-F 2 "Capacitors_SMD:C_1206" H 9550 3900 50  0001 C CNN
-F 3 "" H 9550 3900 50  0000 C CNN
-	1    9550 3900
-	1    0    0    -1
-$EndComp
-Wire Wire Line
-	9550 3600 9550 3800
-Connection ~ 9300 3600
-Wire Wire Line
-	9550 4200 9550 4000
-$Comp
-L GND #PWR071
+L GND #PWR059
 U 1 1 56EDA0C0
 P 2650 3700
-F 0 "#PWR071" H 2650 3450 50  0001 C CNN
+F 0 "#PWR059" H 2650 3450 50  0001 C CNN
 F 1 "GND" H 2650 3550 50  0000 C CNN
 F 2 "" H 2650 3700 50  0000 C CNN
@@
 	4100 3250 4100 4050
 $Comp
-L +5V #PWR?
+L +5V #PWR060
 U 1 1 580F2142
 P 4100 5550
-F 0 "#PWR?" H 4100 5400 50  0001 C CNN
+F 0 "#PWR060" H 4100 5400 50  0001 C CNN
 F 1 "+5V" H 4100 5690 50  0000 C CNN
 F 2 "" H 4100 5550 50  0000 C CNN
@@
 	1    0    0    -1
 $EndComp
+Text Notes 7500 3900 0    60   ~ 0
+uSD card slot has been removed.\n
 $EndSCHEMATC

Commit message: BlackWolf PCB design completed
Connections:
- no-connect marks 0 -> 4
Changed lines of the file:
@@
 Text Notes 7500 3900 0    60   ~ 0
 uSD card slot has been removed.\n
+NoConn ~ 2800 5800
+NoConn ~ 2800 5900
+NoConn ~ 2900 3300
+NoConn ~ 2900 3400
 $EndSCHEMATC
