File: hardware/v2.0-BlackWolf/finder.sch (KiCad schematic (older format))
At the start: 32 parts, among them Q1 DMN3150LW, Q2 DMN3150LW, Q3 DMN3150LW, Q4 DMN3150LW, Q5 TEFT4300, Q6 TEFT4300, Q7 TEFT4300, Q8 TEFT4300

Commit message: PCB: Added IR LED switch line
Connections:
- net EMITTER_SIDES renamed EMITTER_L
- net EMITTER_L: no longer Q3.1 (G), R_F5.1
- new net EMITTER_R: Q3.1 (G), R_F5.1
Changed lines of the file:
@@
 EMITTER_FL
 Connection ~ 1800 3700
-Text HLabel 1550 4450 0    60   Input ~ 0
-EMITTER_SIDES
+Text HLabel 1550 4200 0    60   Input ~ 0
+EMITTER_L
 Connection ~ 2550 4200
 Connection ~ 3300 4700
@@
 EMITTER_FR
 Wire Wire Line
-	1550 4450 1650 4450
+	1550 4200 2600 4200
 Wire Wire Line
-	1650 4200 1650 4700
-Connection ~ 1650 4200
-Connection ~ 1650 4700
-Connection ~ 1650 4450
-Wire Wire Line
-	1650 4200 2600 4200
-Wire Wire Line
-	1650 4700 3350 4700
+	1550 4700 3350 4700
 Text HLabel 6500 3850 2    60   Output ~ 0
 RECV_FL
@@
 Text Notes 6000 2750 0    60   ~ 12
 Soldering Note.\nPhototransistor: Longer pins are emitters (pin 2).
+Text HLabel 1550 4700 0    60   Input ~ 0
+EMITTER_R
 $EndSCHEMATC
